File: EM2.sch (EAGLE design)
At the start: 120 parts, among them IC1 EUP3476SO08T, IC2 APX811-44UG-7, IC3 ATMEGA16U2-MU, IC4 MCP24AA025E48, IC6 W5100SQFP80, IC9 ATMEGA2560-16AU, J1 DC_2_1MM, P1 USB-6PSMT, P3 ICSP:USB, P4 microSD, Q2 2N7002, Q3 2N7002, U1 HY931147C-RJ45, X1 16MHz, X2 25MHz, X3 16MHz

Commit message: Major rework using W5500 ethernet chip
Parts:
- removed C18: 10nF, freetronics-marc:CAP0603
- removed C25, C26, C28: 100nF, freetronics-marc:CAP0603
- removed LED1, LED3, LED9: YELLOW, freetronics-jon:LED0603
- removed LED4: RED, freetronics-jon:LED0603
- removed Q3: 2N7002, freetronics:MOSFET-NCHANNELSMD
- removed RN4: 10K, freetronics-master-v1:4R-NCAY16
- removed RN7: 1K, freetronics-master-v1:4R-NCAY16
- removed SJ4: D2_INT, jumper:SJ
- added C14: 100nF, freetronics-jon:CAP0603
- added C5: 10nF, freetronics-jon:CAP0603
- added R16, R17: 10K 0603, freetronics-marc:RESISTOR0603
- added R22: 10K, freetronics-marc:RESISTOR0603
- added RN9: 1K, freetronics-master-v1.1:4R-NCAY16
- C17: device freetronics-marc:CAP0603 -> freetronics-jon:CAP0603
- C3: value 10uF 6.3V A TANT -> 4.7uF 6.3V A TANT
- IC6: value W5100SQFP80 -> W5500; device freetronics-marc:W5100SQFP80 -> W5500:W5500
- J1: device freetronics:POWER_JACKPTH -> freetronics-jon:POWER_JACKPTH_SLOTS
- L1, L2: value 1uH 250mA 0805 -> Bourns MH2029-300Y 30R 3A 0805
- LED8: value GREEN -> YELLOW
- RN1, RN2: value 1K -> 10K; device freetronics-master-v1:4R-NCAY16 -> freetronics-master-v1.1:4R-NCAY16
- SJ1, SJ3: device jumper:SJ -> freetronics-jon:SJCN
Connections:
- removed net 1V8A: C17.1, C4.+, IC6.VCC1V8A0, IC6.VCC1V8A1, L1.2
- removed net 1V8_OUT: C26.1, C28.1, C3.+, IC6.1V8_OUT, IC6.VCC1V8D0, IC6.VCC1V8D1, IC6.VCC1V8D2, IC6.VCC1V8D3, L1.1
- removed net COLLED: IC6.COLLED, RN1C.1
- removed net D10: IC6./SCS, IC9.(OC2A/PCINT4)PB4, PWMH.3, Q3.G
- removed net N$27: IC6./CS, IC6./RD, IC6./WR, RN7B.1
- removed net N$322: IC6.RSET_BG, R6.2
- removed net N$328: LED4.C, RN1C.2
- removed net N$330: LED1.C, RN1A.2
- removed net N$332: RN2B.1, U1.Y-
- removed net N$67: RN2A.1, U1.G-
- removed net SEN: IC6.SEN, Q3.D, RN7D.1
- removed net WRXLED: IC6.RXLED, RN1B.1
- removed net WTXLED: IC6.TXLED, RN1A.1
- new net 3.3V: C10.+, JP6.5, L1.1, L2.1, LED7.A, LED8.A, REG1.OUT, REG1.OUT@1, REG2.OUT, REG2.OUT@1, U1.G+, U1.Y+
- new net ACTLED: IC6.ACTLED, RN9A.1
- new net D10_SS: IC6.SCS_N, IC9.(OC2A/PCINT4)PB4, PWMH.3, RN2D.1
- new net EXRES1: IC6.EXRES1, R6.2
- new net INT: IC6.INT_N, RN2C.1
- new net N$63: IC6.RSVD@4, RN1C.1
- new net N$73: IC6.RSVD@5, RN1B.1
- new net N$76: IC6.RSVD@6, RN1A.1
- new net N$78: IC6.RSVD@1, R22.2
- new net N$79: IC6.RSVD@2, RN2A.1
- new net N$80: C5.1, IC6.1V2O
- new net N$81: C3.+, IC6.TOCAP
- new net PMODE0: IC6.PMODE0
- new net PMODE1: IC6.PMODE1
- new net PMODE2: IC6.PMODE2
- net 3V3A: now also C14.1, C17.1, C4.+, IC6.AVDD@1, IC6.AVDD@2, IC6.AVDD@3, IC6.AVDD@4, IC6.AVDD@5, IC6.AVDD@6, L1.2; no longer C13.+, C18.1, IC6.VCC3V3A, L2.2
- net 3V3D: now also C13.+, IC6.VDD, L2.2, RN2B.2, RN2C.2, RN2D.2; no longer C10.+, C25.1, IC6.VCC3V3D0, IC6.VCC3V3D1, IC6.VCC3V3D2, JP6.5, L2.1, LED1.A, LED3.A, LED4.A, LED7.A, LED8.A, LED9.A, REG1.OUT, REG1.OUT@1, REG2.OUT, REG2.OUT@1, RN7B.2, RN7D.2, U1.G+, U1.Y+
- net 5V: now also R16.2, R17.2; no longer RN4A.2, RN4B.2
- net D2: no longer SJ4.1
- net FDXLED: now also IC6.DUPLED, RN9B.1; no longer IC6.FDXLED, RN1D.1, RN2A.2
- net GND: now also C14.2, C5.2, IC6.AGND@1, IC6.AGND@2, IC6.AGND@3, IC6.AGND@4, IC6.AGND@5, IC6.AGND@6, IC6.GND, R22.1, RN1A.2, RN1B.2, RN1C.2, RN1D.2, RN2A.2; no longer C18.2, C25.2, C26.2, C28.2, IC6.ADDR0, IC6.ADDR1, IC6.ADDR10, IC6.ADDR11, IC6.ADDR12, IC6.ADDR13, IC6.ADDR14, IC6.ADDR2, IC6.ADDR3, IC6.ADDR4, IC6.ADDR5, IC6.ADDR6, IC6.ADDR7, IC6.ADDR8, IC6.ADDR9, IC6.DATA0, IC6.DATA1, IC6.DATA2, IC6.DATA3, IC6.DATA4, IC6.DATA5, IC6.DATA6, IC6.DATA7, IC6.GNDA0, IC6.GNDA1, IC6.GNDA2, IC6.GNDD0, IC6.GNDD1, IC6.GNDD2, IC6.GNDD3, IC6.GNDD4, IC6.GNDD5, IC6.OPMODE0, IC6.OPMODE1, IC6.OPMODE2, IC6.TEST_MODE0, IC6.TEST_MODE1, IC6.TEST_MODE2, IC6.TEST_MODE3, Q3.S
- net LINKLED: now also RN9C.1; no longer RN2B.2, RN2D.1
- net N$26: now also RN9D.2; no longer RN2C.2
- net N$28: now also RN9C.2, U1.G-; no longer LED9.C, RN2D.2
- net N$327: now also RN9B.2; no longer RN1D.2
- net N$329: now also RN9A.2, U1.Y-; no longer LED3.C, RN1B.2
- net N$62: now also IC6.RSVD@3, RN1D.1; no longer IC6./INT, SJ4.2
- net RESET: now also R16.1; no longer RN4B.1
- net RESET2: now also R17.1; no longer RN4A.1
- net RXIN: now also IC6.RXN; no longer IC6.RXIN
- net RXIP: now also IC6.RXP; no longer IC6.RXIP
- net SPDLED: now also RN9D.1; no longer RN2C.1
- net TXON: now also IC6.TXN; no longer IC6.TXON
- net TXOP: now also IC6.TXP; no longer IC6.TXOP
- net WIZRST: now also IC6.RST_N, RN2B.1; no longer IC6./RESET
- net XTLN: now also C15.1, IC6.XO, R3.1, X2.1; no longer C16.1, IC6.XTLN, R3.2, X2.2
- net XTLP: now also C16.1, IC6.XI/CLKIN, R3.2, X2.2; no longer C15.1, IC6.XTLP, R3.1, X2.1
Other:
- note added: "3.3V Decoupling"
- note added: "ACTIVITY"
- note added: "Freetronics EtherMega2 (Arduino Compatible)"
- note added: "LINK"
- note added: "Note: Leaving PMODE1/2/3 pins floating, because the datasheet says these have internal pull-ups which defaults to the mode being set to auto-negotiate at all possible speeds. Some other Arduino related designs clamp these pins, but it shouldn't be necessary."
- note added: "SKU: EM2"
- note added: "V4.0 (2018-04-16)"
- note added: "Wiznet W5500 Power-On/Reset"
- note added: "www.freetronics.com.au/em2"
- note removed: "1.8V / 3.3V Decoupling"
- note removed: "D2 used if Wiznet Ethernet IC "interrupt" jumper enabled."
- note removed: "SHORT SJ1 and SJ3 on PCB *AFTER* FINAL DRC"
- note removed: "SKU: EM"
- note removed: "SPI D10_SS/nCS low = SEN high = SPI enabled"
- note removed: "SPI MISO tri-state by SS/nCS"
- note removed: "SuperHouse EtherMega (Arduino Compatible)"
- note removed: "V3.1 (2017-12-21)"
- note removed: "Wiznet W5100 Power-On/Reset"
- note removed: "www.superhouse.tv/em"
- moved on the sheet: C13, C15, C16, C17, C3, C4, L1, L2, LED7, LED8, R3, R6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
